File: hardware/kicad/smart-waterer.kicad_sch (KiCad schematic)
At the start: 0 parts

Commit message: fix: 按照空项目正确格式重写原理图
修复:
- 使用用户提供的空项目格式
- 移除 project 和 sheet 块（不需要）
- lib_symbols 保留但添加基本符号
- 保留 title_block, components, nets, wires 等
- 保留 sheet_instances 和 embedded_fonts

格式完全匹配空项目：
(kicad_sch
	(version 20250114)
	(generator "eeschema")
	(generator_version "9.0")
	...
)
Other:
- removed sheet ?
- company: (none) -> Smart Waterer Team
- title: (none) -> 智能浇花机 v0.4（简化版）

Commit message: fix: 使用制表符缩进，完全匹配空项目格式
修复:
- 第一行：(kicad_sch
- 所有制表符使用 tab（^I）
- 完全匹配空项目格式
- 添加所有产品元件
Other:
- title: 智能浇花机 v0.4（简化版） -> 智能浇花机 v0.4
Changed lines of the file:
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@@
 	(paper "A4")
 	(title_block
-		(title "智能浇花机 v0.4（简化版）")
+		(title "智能浇花机 v0.4")
 		(date "2026-03-13")
 		(rev "v0.4")
