File: hardware/kicad/smart-waterer.kicad_sch (KiCad schematic)
At the start: 0 parts

Commit message: fix: 将 components 改为 symbol 顶层结构
Parts:
- added C1: 100nF, Capacitor_SMD:C_0805, symbol Device:C
- added D1: SMAJ5.0A, Diode_SMD:D_SMA, symbol Device:D
- added D2: 1N4007, Diode_SMD:D_SOD-323, symbol Device:D
- added F1: 1812L110, Fuse:Fuse_1812, symbol Device:Fuse
- added J1: USB-C, Connector_USB:USB_C_Receptacle, symbol Connector:USB_C_Receptacle
- added J2: 土壤湿度, TerminalBlock:TerminalBlock_KF301-2P, symbol Connector:TerminalBlock_KF301-2P
- added J3: 水位检测, TerminalBlock:TerminalBlock_KF301-2P, symbol Connector:TerminalBlock_KF301-2P
- added J4: 水泵, TerminalBlock:TerminalBlock_KF301-2P, symbol Connector:TerminalBlock_KF301-2P
- added J5: NTC, TerminalBlock:TerminalBlock_KF301-2P, symbol Connector:TerminalBlock_KF301-2P
- added Q1: AO4606, Package_SO:SOIC-8, symbol Device:Q_NJFET_GSD
- added R1: 10kΩ, Resistor_SMD:R_0805, symbol Device:R
- added TH1: NTC 10kΩ B3950, Resistor_SMD:R_0805, symbol Device:R
- added U1: ESP32-C3-SuperMini, ESP32-C3-SuperMini, symbol ESP32-C3-SuperMini
- added U2: XC6206-3.3V, Package_TO_SOT_SMD:SOT-23, symbol Regulator_Linear:XC6206-3.3V
- added U3: TP4056, Package_DFN_QFN:DFN-8, symbol Charger:TP4056
- added U4: MT3608, Package_TO_SOT_SMD:SOT-23-6, symbol Regulator_Switching:MT3608
Connections:
- no-connect marks 0 -> 2
